File: board/kachisys.sch (EAGLE design)
At the start: 88 parts, among them IC1 LT1963ES8-3.3, J1 S3B-PH-SM4-TB(LF)(SN), J2 S3B-PH-SM4-TB(LF)(SN), J3 S3B-PH-SM4-TB(LF)(SN), J4 S3B-PH-SM4-TB(LF)(SN), J5 S3B-PH-SM4-TB(LF)(SN), J6 S3B-PH-SM4-TB(LF)(SN), J7 S3B-PH-SM4-TB(LF)(SN), J8 ZX62R-AB-5P, J9 2DC-0415D200, SW1 EN_SW, SW2 IO0_SW, T1 MMSS8050, T2 MMSS8050, U1 FT231XS, U2 ESP-WROOM-32, U3 BME280

Commit message: rev.2 upload
Parts:
- removed IC1: LT1963ES8-3.3, linear-technology:LT1963ES8-3.3
- added U4: ADP3338AKCZ-3.3, taki-library:ADP3338AKCZ-3.3
Connections:
- net +3V3: now also U4.OUT; no longer IC1G$1.OUT, IC1G$1.SENSE
- net +5V: now also U4.IN; no longer IC1G$1.!SHDN, IC1G$1.IN
- net GND: now also U4.GND; no longer IC1G$1.GND
Changed lines of the file:
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@@
 <part name="C1" library="resistor" library_urn="urn:adsk.eagle:library:348" deviceset="C-EU" device="C2012" package3d_urn="urn:adsk.eagle:package:23625/2" value="22μF"/>
 <part name="U1" library="SparkFun-IC-Comms" library_urn="urn:adsk.eagle:library:521" deviceset="FT231X" device="S" package3d_urn="urn:adsk.eagle:package:38726/1" value="FT231XS"/>
-<part name="IC1" library="linear-technology" library_urn="urn:adsk.eagle:library:261" deviceset="LT1963ES8" device="" package3d_urn="urn:adsk.eagle:package:16057/1" technology="-3.3"/>
 <part name="C2" library="resistor" library_urn="urn:adsk.eagle:library:348" deviceset="C-EU" device="C2012" package3d_urn="urn:adsk.eagle:package:23625/2" value="22μF"/>
 <part name="+3V1" library="supply1" library_urn="urn:adsk.eagle:library:371" deviceset="+3V3" device=""/>
@@
 <part name="GND31" library="180118 Library by matsu" library_urn="urn:adsk.eagle:library:5572060" deviceset="GND" device=""/>
 <part name="GND32" library="180118 Library by matsu" library_urn="urn:adsk.eagle:library:5572060" deviceset="GND" device=""/>
+<part name="U4" library="taki-library" deviceset="ADP3338AKCZ-3.3" device=""/>
 </parts>
 <sheets>
@@
 <instance part="R8" gate="G$1" x="-83.82" y="-83.82" rot="R180"/>
 <instance part="C1" gate="G$1" x="111.76" y="68.58"/>
-<instance part="IC1" gate="G$1" x="129.54" y="71.12"/>
 <instance part="C2" gate="G$1" x="147.32" y="68.58"/>
 <instance part="+3V4" gate="G$1" x="162.56" y="83.82"/>
@@
 <instance part="GND31" gate="1" x="-88.9" y="-154.94"/>
 <instance part="GND32" gate="1" x="-78.74" y="-154.94"/>
+<instance part="U4" gate="A" x="129.54" y="73.66"/>
 </instances>
 <busses>
@@
 <wire x1="147.32" y1="50.8" x2="147.32" y2="63.5" width="0.1524" layer="91"/>
 <pinref part="GND16" gate="1" pin="GND"/>
-</segment>
-<segment>
-<pinref part="IC1" gate="G$1" pin="GND"/>
-<wire x1="129.54" y1="50.8" x2="129.54" y2="60.96" width="0.1524" layer="91"/>
-<pinref part="GND17" gate="1" pin="GND"/>
 </segment>
 <segment>
@@
 <wire x1="-78.74" y1="-144.78" x2="-78.74" y2="-152.4" width="0.1524" layer="91"/>
 <pinref part="GND32" gate="1" pin="GND"/>
+</segment>
+<segment>
+<pinref part="U4" gate="A" pin="GND"/>
+<pinref part="GND17" gate="1" pin="GND"/>
+<wire x1="129.54" y1="60.96" x2="129.54" y2="50.8" width="0.1524" layer="91"/>
 </segment>
 </net>
@@
 </segment>
 <segment>
-<pinref part="IC1" gate="G$1" pin="OUT"/>
-<wire x1="139.7" y1="73.66" x2="142.24" y2="73.66" width="0.1524" layer="91"/>
-<pinref part="IC1" gate="G$1" pin="SENSE"/>
-<wire x1="142.24" y1="73.66" x2="144.78" y2="73.66" width="0.1524" layer="91"/>
-<wire x1="139.7" y1="71.12" x2="142.24" y2="71.12" width="0.1524" layer="91"/>
-<wire x1="142.24" y1="71.12" x2="142.24" y2="73.66" width="0.1524" layer="91"/>
-<junction x="142.24" y="73.66"/>
-<wire x1="144.78" y1="73.66" x2="147.32" y2="73.66" width="0.1524" layer="91"/>
 <pinref part="C2" gate="G$1" pin="1"/>
 <wire x1="147.32" y1="73.66" x2="162.56" y2="73.66" width="0.1524" layer="91"/>
 <wire x1="147.32" y1="73.66" x2="147.32" y2="71.12" width="0.1524" layer="91"/>
-<junction x="147.32" y="73.66"/>
 <pinref part="+3V4" gate="G$1" pin="+3V3"/>
 <wire x1="162.56" y1="73.66" x2="162.56" y2="81.28" width="0.1524" layer="91"/>
@@
 <pinref part="R9" gate="G$1" pin="2"/>
 <wire x1="162.56" y1="71.12" x2="162.56" y2="73.66" width="0.1524" layer="91"/>
+<pinref part="U4" gate="A" pin="OUT"/>
+<wire x1="142.24" y1="73.66" x2="147.32" y2="73.66" width="0.1524" layer="91"/>
+<junction x="147.32" y="73.66"/>
 </segment>
 <segment>
@@
 </segment>
 <segment>
-<pinref part="IC1" gate="G$1" pin="IN"/>
-<wire x1="111.76" y1="73.66" x2="116.84" y2="73.66" width="0.1524" layer="91"/>
-<wire x1="116.84" y1="73.66" x2="119.38" y2="73.66" width="0.1524" layer="91"/>
-<pinref part="IC1" gate="G$1" pin="!SHDN"/>
-<wire x1="119.38" y1="68.58" x2="116.84" y2="68.58" width="0.1524" layer="91"/>
-<wire x1="116.84" y1="68.58" x2="116.84" y2="73.66" width="0.1524" layer="91"/>
-<junction x="116.84" y="73.66"/>
 <pinref part="C1" gate="G$1" pin="1"/>
 <wire x1="111.76" y1="71.12" x2="111.76" y2="73.66" width="0.1524" layer="91"/>
 <wire x1="111.76" y1="73.66" x2="101.6" y2="73.66" width="0.1524" layer="91"/>
-<junction x="111.76" y="73.66"/>
 <wire x1="101.6" y1="73.66" x2="101.6" y2="81.28" width="0.1524" layer="91"/>
 <pinref part="P+7" gate="1" pin="+5V"/>
-</segment>
-</net>
+<pinref part="U4" gate="A" pin="IN"/>
+<wire x1="116.84" y1="73.66" x2="111.76" y2="73.66" width="0.1524" layer="91"/>
+<junction x="111.76" y="73.66"/>
+</segment>
+</net>
