File: board/kachisys.brd (EAGLE design)
At the start: 100 x 83 mm, 88 parts, among them IC1 LT1963ES8-3.3, J1 S3B-PH-SM4-TB(LF)(SN), J2 S3B-PH-SM4-TB(LF)(SN), J3 S3B-PH-SM4-TB(LF)(SN), J4 S3B-PH-SM4-TB(LF)(SN), J5 S3B-PH-SM4-TB(LF)(SN), J6 S3B-PH-SM4-TB(LF)(SN), J7 S3B-PH-SM4-TB(LF)(SN), J8 ZX62R-AB-5P, J9 2DC-0415D200, SW1 EN_SW, SW2 IO0_SW, T1 MMSS8050, T2 MMSS8050, U1 FT231XS, U2 ESP-WROOM-32, U3 BME280

Commit message: rev.2 upload
Parts:
- removed IC1: LT1963ES8-3.3, linear-technology:SOIC8
- added U4: ADP3338AKCZ-3.3, taki-library:SOT233
- moved C3 19.1 mm to (5.00, -4.00), turned to 0 degrees
- moved J9 17.4 mm to (14.0, -19.0), turned to 90 degrees
- moved J8 12.6 mm to (86.0, -17.5), turned to 0 degrees
- moved C1 5.64 mm to (24.4, -6.84), turned to 270 degrees
- moved C2 2.94 mm to (35.7, -2.67), turned to 270 degrees
- moved C20 2.00 mm to (17.0, 0.00)
- flipped C13 to the bottom
- flipped U3 to the bottom, turned to 270 degrees
Connections:
- net +3V3: now also U4.2, U4.4; no longer IC1.1, IC1.2
- net +5V: now also U4.3; no longer IC1.5, IC1.8
- net GND: now also U4.1; no longer IC1.3, IC1.6, IC1.7
Routing:
- net GND: track 129.9 -> 604.0 mm, vias 10 -> 37
- net +5V: track 406.1 -> 393.2 mm
- net +3V3: track 273.8 -> 286.1 mm, vias 7 -> 9
- net N$2: track 21.2 -> 10.8 mm
- net N$3: track 19.3 -> 10.4 mm
- net IO32: track 35.4 -> 40.2 mm
- net IO23: track 65.2 -> 69.6 mm
- net N$5: track 19.6 -> 16.9 mm, vias 3 -> 2
- net N$4: track 21.7 -> 20.2 mm
- net EN: track 114.4 -> 115.6 mm
- net IO33: track 35.5 -> 36.6 mm
- net IO21: track 64.5 -> 63.9 mm
- net N$46: track 14.2 -> 13.6 mm
- net IO16: track 60.2 -> 59.6 mm
- net N$40: track 14.9 -> 14.4 mm
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- added copper zone on layer 1, net GND
Other:
- board size 100 x 83 mm -> 100 x 62 mm
- board text added: "1"
- board text added: "Kachi-sys for NITTC Procon Semi Room Designed by Kapipara 2018/12/01 rev.2"
- board text removed: "Kachi-sys for NITTC Procon Semi Room Designed by Kapipara 2018/10/01 rev.1"

Commit message: garv修正，謎のAirwire修正
Routing:
- net GND: track 604.0 -> 606.6 mm
Changed lines of the file:
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@@
 <wire x1="24" y1="8.1" x2="26.13" y2="8.1" width="0.75" layer="16"/>
 <wire x1="33.73" y1="8.1" x2="35.7" y2="8.1" width="0.75" layer="16"/>
-<polygon width="0" layer="16" isolate="0.4">
-<vertex x="-1" y="44"/>
-<vertex x="101" y="44"/>
-<vertex x="101" y="-20"/>
-<vertex x="-1" y="-20"/>
-</polygon>
 <wire x1="35.7" y1="8.1" x2="37.88" y2="8.1" width="0.75" layer="16"/>
 <wire x1="15.2" y1="37.7" x2="14.5" y2="37.7" width="0.75" layer="1"/>
@@
 <wire x1="82.9" y1="-15.15" x2="81.9" y2="-16.15" width="0.75" layer="16"/>
 <wire x1="81.9" y1="-16.15" x2="81.9" y2="-17.5" width="0.75" layer="16"/>
-<wire x1="81.25" y1="-10.5" x2="81.25" y2="-11.25" width="0.75" layer="16"/>
 <wire x1="86.2275" y1="-10.5" x2="86.2275" y2="-8.7725" width="0.75" layer="16"/>
 <wire x1="88" y1="-7" x2="91.5" y2="-7" width="0.75" layer="16"/>
@@
 <wire x1="89" y1="25" x2="89" y2="27" width="0.75" layer="1"/>
 <wire x1="83.9" y1="24" x2="88" y2="24" width="0.75" layer="1"/>
-<polygon width="0" layer="1" isolate="0.4">
-<vertex x="-2" y="45"/>
-<vertex x="102" y="45"/>
-<vertex x="102" y="-21"/>
-<vertex x="-2" y="-21"/>
-</polygon>
 <wire x1="87.3" y1="-14.825" x2="87.3" y2="-12.6774" width="0.4" layer="16"/>
 <wire x1="87.3" y1="-12.6774" x2="87.3774" y2="-12.6774" width="0.4" layer="16"/>
@@
 <via x="55.8" y="-4.8" extent="1-16" drill="0.35"/>
 <wire x1="55.8" y1="-4.8" x2="54.4" y2="-4.8" width="0.75" layer="16"/>
-<wire x1="82.9" y1="-13.1" x2="82.9" y2="-15.15" width="0.75" layer="16"/>
-<wire x1="81.25" y1="-11.25" x2="81.25" y2="-11.25" width="0.75" layer="16"/>
+<wire x1="81.25" y1="-10.5" x2="81.25" y2="-11.25" width="0.75" layer="16"/>
+<wire x1="81.25" y1="-11.25" x2="83" y2="-13" width="0.75" layer="16"/>
+<wire x1="83" y1="-13" x2="83" y2="-15.05" width="0.75" layer="16"/>
+<wire x1="83" y1="-15.05" x2="82.925" y2="-15.125" width="0.75" layer="16"/>
+<wire x1="82.925" y1="-15.125" x2="82.9" y2="-15.125" width="0.75" layer="16"/>
+<polygon width="0.2" layer="1" isolate="0.4">
+<vertex x="0" y="43"/>
+<vertex x="100" y="43"/>
+<vertex x="100" y="-19"/>
+<vertex x="0" y="-19"/>
+</polygon>
+<polygon width="0.2" layer="16" isolate="0.4">
+<vertex x="0" y="43"/>
+<vertex x="100" y="43"/>
+<vertex x="100" y="-19"/>
+<vertex x="0" y="-19"/>
+</polygon>
 </signal>
 <signal name="+3V3" class="1">
